File: kicad/LR1120_Mikrobus/_autosave-LR1120_Mikrobus.kicad_sch (KiCad schematic)
At the start: 82 parts, among them Q1 NX2016SA-32M-EXS00A-CS06465, Q2 NT2016SA-32M-END4263A, Q3 NX3215SA, U1 LR1120, U2 SKY13588-460LF, U5 LIS2DE12, U7 M24128-BFMH6TG, U8 BGA524N6E6327XTSA1

Commit message: All changes
Parts:
- C11, C16, C20: value 0.5pF -> NC
- C14: value 0.5pF -> 6.8pF
- C52: value 100nF -> NC; footprint Capacitor_SMD:C_0201_0603Metric_Pad0.64x0.40mm_HandSolder -> Capacitor_SMD:C_0201_0603Metric
Changed lines of the file:
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@@
     (in_bom yes) (on_board yes)
     (property "Reference" "C16" (id 0) (at 40.64 60.96 0))
-    (property "Value" "0.5pF" (id 1) (at 40.64 55.88 0))
+    (property "Value" "NC" (id 1) (at 40.64 55.88 0))
     (property "Footprint" "Capacitor_SMD:C_01005_0402Metric" (id 2) (at 45.4152 62.23 0)
       (effects (font (size 1.27 1.27)) hide)
@@
     (in_bom yes) (on_board yes)
     (property "Reference" "C14" (id 0) (at 57.15 60.96 0))
-    (property "Value" "0.5pF" (id 1) (at 57.15 55.88 0))
+    (property "Value" "6.8pF" (id 1) (at 57.15 55.88 0))
     (property "Footprint" "Capacitor_SMD:C_01005_0402Metric" (id 2) (at 61.9252 62.23 0)
       (effects (font (size 1.27 1.27)) hide)
@@
       (effects (font (size 1.27 1.27)) (justify left))
     )
-    (property "Value" "100nF" (id 1) (at 242.57 133.3499 0)
-      (effects (font (size 1.27 1.27)) (justify left))
-    )
-    (property "Footprint" "Capacitor_SMD:C_0201_0603Metric_Pad0.64x0.40mm_HandSolder" (id 2) (at 239.7252 135.89 0)
+    (property "Value" "NC" (id 1) (at 242.57 133.3499 0)
+      (effects (font (size 1.27 1.27)) (justify left))
+    )
+    (property "Footprint" "Capacitor_SMD:C_0201_0603Metric" (id 2) (at 239.7252 135.89 0)
       (effects (font (size 1.27 1.27)) hide)
     )
@@
     (in_bom yes) (on_board yes)
     (property "Reference" "C20" (id 0) (at 148.59 49.53 90))
-    (property "Value" "0.5pF" (id 1) (at 153.67 49.53 90))
+    (property "Value" "NC" (id 1) (at 153.67 49.53 90))
     (property "Footprint" "Capacitor_SMD:C_01005_0402Metric" (id 2) (at 147.32 54.3052 0)
       (effects (font (size 1.27 1.27)) hide)
@@
     (in_bom yes) (on_board yes)
     (property "Reference" "C11" (id 0) (at 40.64 83.82 0))
-    (property "Value" "0.5pF" (id 1) (at 40.64 78.74 0))
+    (property "Value" "NC" (id 1) (at 40.64 78.74 0))
     (property "Footprint" "Capacitor_SMD:C_01005_0402Metric" (id 2) (at 45.4152 85.09 0)
       (effects (font (size 1.27 1.27)) hide)
@@
     )
     (path "/ff7778df-5093-417b-82dd-c475f5c81cdc"
-      (reference "C11") (unit 1) (value "0.5pF") (footprint "Capacitor_SMD:C_01005_0402Metric")
+      (reference "C11") (unit 1) (value "NC") (footprint "Capacitor_SMD:C_01005_0402Metric")
     )
     (path "/0d87a121-a86b-4749-8c7b-4b6deea2ee47"
@@
     )
     (path "/7d8c6ac7-884e-467c-8d84-eaa4ae7d9f63"
-      (reference "C14") (unit 1) (value "0.5pF") (footprint "Capacitor_SMD:C_01005_0402Metric")
+      (reference "C14") (unit 1) (value "6.8pF") (footprint "Capacitor_SMD:C_01005_0402Metric")
     )
     (path "/bc4dd6e4-4df9-4089-8b74-6267bfdb1080"
@@
     )
     (path "/5f55865b-0b6e-4cb8-a110-73d5d0793886"
-      (reference "C16") (unit 1) (value "0.5pF") (footprint "Capacitor_SMD:C_01005_0402Metric")
+      (reference "C16") (unit 1) (value "NC") (footprint "Capacitor_SMD:C_01005_0402Metric")
     )
     (path "/4fee6e29-04f6-4d2b-8028-17eb5dd0c81c"
@@
     )
     (path "/e5a7a84f-0122-4ef6-8f51-3ec88e85c1a3"
-      (reference "C20") (unit 1) (value "0.5pF") (footprint "Capacitor_SMD:C_01005_0402Metric")
+      (reference "C20") (unit 1) (value "NC") (footprint "Capacitor_SMD:C_01005_0402Metric")
     )
     (path "/7355a802-4b21-400b-899d-c0d47a30cceb"
@@
     )
     (path "/dbb15a35-644e-4998-9510-39d4f76d0325"
-      (reference "C52") (unit 1) (value "100nF") (footprint "Capacitor_SMD:C_0201_0603Metric_Pad0.64x0.40mm_HandSolder")
+      (reference "C52") (unit 1) (value "NC") (footprint "Capacitor_SMD:C_0201_0603Metric")
     )
     (path "/20924966-d251-4062-bd99-6a0a4e9003bc"
